File: TOM2015/Hardware/Interruptor/esp-tom.brd (EAGLE design)
At the start: 93 x 43 mm, 20 parts, among them K1 G5L, X1 MKDSN1,5/2-5,08, X2 MKDSN1,5/3-5,08

Commit message: Versão final do tom
Versão final do Tom com as ligações do esp corretas e o desenho correto
do componente TIL111
Parts:
- OK1: device optocoupler:DIL06 -> optocoupler2:DIL06
- moved U$1 3.66 mm to (77.7, 35.3), turned to 270 degrees
Connections:
- net 3.3V: now also U$1.GPIO2, U$1.VCC; no longer U$1.GPIO0, U$1.TX
- net GND: now also U$1.GND; no longer U$1.RX
- net GPIO0: now also U$1.GPIO0; no longer U$1.GPIO2
Routing:
- net 3.3V: track 58.2 -> 51.4 mm
- net GND: track 39.0 -> 32.7 mm
- net GPIO0: track 51.4 -> 52.6 mm
Changed lines of the file:
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@@
 <attribute name="SPICEPREFIX" value="L" x="52.93" y="34.2" size="1.778" layer="27" rot="R90" display="off"/>
 </element>
-<element name="OK1" library="optocoupler" package="DIL06" value="H11L1M" x="34.32" y="34.15" rot="R90">
+<element name="OK1" library="optocoupler2" package="DIL06" value="H11L1M" x="34.32" y="34.15" rot="R90">
 <attribute name="OC_FARNELL" value="1021127" x="34.32" y="34.15" size="1.778" layer="27" rot="R90" display="off"/>
 <attribute name="MPN" value="H11L1-M" x="34.32" y="34.15" size="1.778" layer="27" rot="R90" display="off"/>
@@
 <element name="R3" library="resistor" package="0204/7" value="47k" x="24.07" y="32.9" rot="R90"/>
 <element name="R4" library="resistor" package="0204/7" value="68k" x="18.11" y="35.76" rot="R270"/>
-<element name="U$1" library="esp8266modules" package="ESP01" value="ESP01" x="81.3" y="34.68" rot="R90"/>
+<element name="U$1" library="esp8266modules" package="ESP01" value="ESP01" x="77.7" y="35.32" rot="R270"/>
 <element name="U$2" library="mylibrary" package="NA03-T2S05" value="NA03-T2S05" x="54.96" y="7.27"/>
 <element name="X1" library="con-phoenix-508" package="MKDSN1,5/2-5,08" value="MKDSN1,5/2-5,08" x="49.56" y="5.99" rot="R270"/>
@@
 <contactref element="R1" pad="2"/>
 <contactref element="R2" pad="2"/>
-<contactref element="U$1" pad="CH_PD"/>
 <contactref element="C3" pad="+"/>
 <contactref element="C4" pad="1"/>
 <contactref element="C5" pad="1"/>
 <contactref element="L3" pad="2"/>
-<contactref element="U$1" pad="RST"/>
 <wire x1="44.09" y1="39.21" x2="48.07" y2="39.19" width="0.8128" layer="16"/>
-<contactref element="U$1" pad="GPIO0"/>
-<contactref element="U$1" pad="TX"/>
-<wire x1="86.9375" y1="35.935" x2="89.4775" y2="35.935" width="0.8128" layer="16"/>
-<wire x1="89.4775" y1="35.935" x2="89.4775" y2="33.395" width="0.8128" layer="16"/>
-<wire x1="89.4775" y1="33.395" x2="89.4775" y2="30.855" width="0.8128" layer="16"/>
-<wire x1="86.9375" y1="35.935" x2="81.45" y2="35.99" width="0.8128" layer="16"/>
-<wire x1="81.45" y1="35.99" x2="76.96" y2="36.01" width="0.8128" layer="16"/>
 <wire x1="48.07" y1="39.19" x2="51" y2="39.19" width="0.8128" layer="16"/>
 <wire x1="51" y1="39.19" x2="51" y2="36" width="0.8128" layer="16"/>
 <wire x1="51" y1="36" x2="57.02" y2="36" width="0.8128" layer="16"/>
 <wire x1="57.02" y1="36" x2="60.5" y2="36" width="0.8128" layer="16"/>
-<wire x1="60.5" y1="36" x2="76.96" y2="36" width="0.8128" layer="16"/>
-<wire x1="76.96" y1="36" x2="76.96" y2="36.01" width="0.8128" layer="16"/>
 <wire x1="57.11" y1="38.58" x2="57.02" y2="36" width="0.8128" layer="16"/>
 <wire x1="60.38" y1="37.924" x2="60.5" y2="36" width="0.8128" layer="16"/>
+<contactref element="U$1" pad="CH_PD"/>
+<contactref element="U$1" pad="VCC"/>
+<contactref element="U$1" pad="RST"/>
+<contactref element="U$1" pad="GPIO2"/>
+<wire x1="69.5225" y1="36.605" x2="69.5225" y2="36" width="0.8128" layer="16"/>
+<wire x1="69.5225" y1="36" x2="60.5" y2="36" width="0.8128" layer="16"/>
+<wire x1="69.5225" y1="31.525" x2="69.5225" y2="34.065" width="0.8128" layer="16"/>
+<wire x1="69.5225" y1="34.065" x2="69.5225" y2="36.605" width="0.8128" layer="16"/>
+<wire x1="69.5225" y1="36.605" x2="72.0625" y2="36.605" width="0.8128" layer="16"/>
+<wire x1="72.0625" y1="36.605" x2="72.0625" y2="36.01" width="0.8128" layer="16"/>
+<wire x1="72.0625" y1="36.01" x2="76.96" y2="36.01" width="0.8128" layer="16"/>
+<wire x1="76.96" y1="36.01" x2="76.96" y2="35.99" width="0.8128" layer="16"/>
+<wire x1="76.96" y1="35.99" x2="81.45" y2="35.99" width="0.8128" layer="16"/>
 </signal>
 <signal name="GPIO0">
@@
 <contactref element="R2" pad="1"/>
 <wire x1="38.13" y1="34.15" x2="48.07" y2="34.15" width="0.8128" layer="16"/>
-<wire x1="48.07" y1="33.395" x2="48.07" y2="31.57" width="0.8128" layer="16"/>
-<contactref element="U$1" pad="GPIO2"/>
-<wire x1="86.9375" y1="33.395" x2="48.07" y2="33.395" width="0.8128" layer="16"/>
-<wire x1="48.07" y1="33.395" x2="48.07" y2="34.15" width="0.8128" layer="16"/>
+<wire x1="48.07" y1="34.15" x2="48.07" y2="31.57" width="0.8128" layer="16"/>
+<contactref element="U$1" pad="GPIO0"/>
+<wire x1="48.07" y1="34.15" x2="48.07" y2="34.16" width="0.8128" layer="16"/>
+<wire x1="48.07" y1="34.16" x2="67.58" y2="34.16" width="0.8128" layer="16"/>
+<wire x1="67.58" y1="34.16" x2="67.56" y2="29" width="0.8128" layer="16"/>
+<wire x1="67.56" y1="29" x2="75" y2="29" width="0.8128" layer="16"/>
+<wire x1="75" y1="29" x2="75" y2="34.065" width="0.8128" layer="16"/>
+<wire x1="75" y1="34.065" x2="72.0625" y2="34.065" width="0.8128" layer="16"/>
 </signal>
 <signal name="N$2">
@@
 <wire x1="60.38" y1="39.956" x2="52.93" y2="39.956" width="0.8128" layer="16"/>
 <wire x1="52.93" y1="39.956" x2="52.93" y2="39.28" width="0.8128" layer="16"/>
-<contactref element="U$1" pad="RX"/>
-<wire x1="60.38" y1="39.956" x2="76.98" y2="39.956" width="0.8128" layer="16"/>
-<wire x1="76.98" y1="39.956" x2="81.48" y2="39.956" width="0.8128" layer="16"/>
-<wire x1="81.48" y1="39.956" x2="86.9375" y2="39.956" width="0.8128" layer="16"/>
-<wire x1="86.9375" y1="39.956" x2="86.9375" y2="38.475" width="0.8128" layer="16"/>
-<wire x1="76.96" y1="38.55" x2="76.98" y2="39.956" width="0.8128" layer="16"/>
-<wire x1="81.45" y1="38.53" x2="81.48" y2="39.956" width="0.8128" layer="16"/>
+<contactref element="U$1" pad="GND"/>
+<wire x1="60.38" y1="39.956" x2="60.38" y2="41" width="0.8128" layer="16"/>
+<wire x1="60.38" y1="41" x2="72" y2="41" width="0.8128" layer="16"/>
+<wire x1="72" y1="41" x2="72" y2="39.145" width="0.8128" layer="16"/>
+<wire x1="72" y1="39.145" x2="72.0625" y2="39.145" width="0.8128" layer="16"/>
+<wire x1="72.0625" y1="39.145" x2="72.0625" y2="38.55" width="0.8128" layer="16"/>
+<wire x1="72.0625" y1="38.55" x2="76.96" y2="38.55" width="0.8128" layer="16"/>
+<wire x1="76.96" y1="38.55" x2="76.96" y2="38.53" width="0.8128" layer="16"/>
+<wire x1="76.96" y1="38.53" x2="81.45" y2="38.53" width="0.8128" layer="16"/>
 </signal>
 <signal name="N$4">
