File: TOM2015/Hardware/Tomada/tomada esp-tom.brd (EAGLE design)
At the start: 52 x 65 mm, 20 parts, among them K2 G5L, X1 MKDSN1,5/2-5,08, X2 MKDSN1,5/2-5,08

Commit message: Versão final do tom
Versão final do Tom com as ligações do esp corretas e o desenho correto
do componente TIL111
Parts:
- OK1: device optocoupler:DIL06 -> optocoupler2:DIL06
- moved C5 7.60 mm to (38.0, 5.72), turned to 270 degrees
- moved C4 6.10 mm to (41.5, 5.74), turned to 270 degrees
- moved R1 5.00 mm to (35.1, 5.34)
- moved R2 4.76 mm to (38.6, 12.1), turned to 180 degrees
Connections:
- net 3.3V: now also U$1.GPIO2, U$1.VCC; no longer U$1.GPIO0, U$1.TX
- net GND: now also U$1.GND; no longer U$1.RX
- net GPIO0: now also U$1.GPIO0; no longer U$1.GPIO2
Routing:
- net GND: track 34.2 -> 67.3 mm
- net 3.3V: track 58.0 -> 44.8 mm
- net GPIO0: track 27.6 -> 34.7 mm
- net N$1: track 24.0 -> 19.0 mm
Changed lines of the file:
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@@
 <element name="C2" library="rcl" package="E2-5" value="0.33 uF" x="40.94" y="38.95" rot="R90"/>
 <element name="C3" library="rcl" package="E2-5" value="0.01 uF" x="42.06" y="22.38" rot="R180"/>
-<element name="C4" library="rcl" package="C025-024X044" value="10 uF" x="37.45" y="10.26" rot="R90"/>
-<element name="C5" library="rcl" package="C025-024X044" value="0.1 uF" x="31.96" y="10.28" rot="R90"/>
+<element name="C4" library="rcl" package="C025-024X044" value="10 uF" x="41.55" y="5.74" rot="R270"/>
+<element name="C5" library="rcl" package="C025-024X044" value="0.1 uF" x="38.04" y="5.72" rot="R270"/>
 <element name="D1" library="diode" package="DO41-10" value="1N4004" x="6.2" y="29.85"/>
 <element name="IC1" library="v-reg" package="78LXX" value="" x="46.85" y="39.99" rot="R90"/>
@@
 <attribute name="SPICEPREFIX" value="L" x="36.07" y="30.8" size="1.778" layer="27" rot="R270" display="off"/>
 </element>
-<element name="OK1" library="optocoupler" package="DIL06" value="H11L1M" x="18.32" y="10.15" rot="R90">
+<element name="OK1" library="optocoupler2" package="DIL06" value="H11L1M" x="18.32" y="10.15" rot="R90">
 <attribute name="OC_FARNELL" value="1021127" x="18.32" y="10.15" size="1.778" layer="27" rot="R90" display="off"/>
 <attribute name="MPN" value="H11L1-M" x="18.32" y="10.15" size="1.778" layer="27" rot="R90" display="off"/>
@@
 </element>
 <element name="Q1" library="transistors" package="TO-92" value="" x="6.03" y="22.97" rot="R270"/>
-<element name="R1" library="resistor" package="0204/7" value="330" x="40.12" y="5.34" rot="R90"/>
-<element name="R2" library="resistor" package="0204/7" value="10k" x="43.07" y="10.38" rot="R90"/>
+<element name="R1" library="resistor" package="0204/7" value="330" x="35.12" y="5.34" rot="R90"/>
+<element name="R2" library="resistor" package="0204/7" value="10k" x="38.62" y="12.07" rot="R180"/>
 <element name="R3" library="resistor" package="0204/7" value="47k" x="10.43" y="19.15" rot="R270"/>
 <element name="R4" library="resistor" package="0204/7" value="68k" x="21.01" y="26.81" rot="R270"/>
@@
 <contactref element="OK1" pad="1"/>
 <wire x1="22.13" y1="7.61" x2="22.13" y2="1.59" width="0.8128" layer="16"/>
-<wire x1="22.13" y1="1.59" x2="40.12" y2="1.53" width="0.8128" layer="16"/>
+<wire x1="22.13" y1="1.59" x2="35.12" y2="1.53" width="0.8128" layer="16"/>
 </signal>
 <signal name="3.3V">
 <contactref element="R1" pad="2"/>
 <contactref element="R2" pad="2"/>
-<contactref element="U$1" pad="CH_PD"/>
 <contactref element="C3" pad="+"/>
 <contactref element="C4" pad="1"/>
 <contactref element="C5" pad="1"/>
 <contactref element="L3" pad="2"/>
-<contactref element="U$1" pad="RST"/>
-<contactref element="U$1" pad="GPIO0"/>
-<contactref element="U$1" pad="TX"/>
 <wire x1="46.89" y1="25.42" x2="46.89" y2="22.38" width="0.8128" layer="16"/>
 <wire x1="46.89" y1="22.38" x2="46" y2="22.38" width="0.8128" layer="16"/>
 <wire x1="46" y1="22.38" x2="43.076" y2="22.38" width="0.8128" layer="16"/>
-<wire x1="43.076" y1="22.38" x2="43.076" y2="14.19" width="0.8128" layer="16"/>
-<wire x1="43.076" y1="14.19" x2="43.07" y2="14.19" width="0.8128" layer="16"/>
-<wire x1="43.07" y1="14.19" x2="43.07" y2="13.91" width="0.8128" layer="16"/>
-<wire x1="48.4775" y1="8.935" x2="50.98" y2="8.935" width="0.8128" layer="16"/>
-<wire x1="50.98" y1="8.935" x2="50.98" y2="22.43" width="0.8128" layer="16"/>
-<wire x1="50.98" y1="22.43" x2="46" y2="22.43" width="0.8128" layer="16"/>
 <wire x1="46" y1="22.43" x2="46" y2="22.38" width="0.8128" layer="16"/>
-<wire x1="31.96" y1="9.01" x2="31.96" y2="8.99" width="0.8128" layer="16"/>
-<wire x1="31.96" y1="8.99" x2="37.45" y2="8.99" width="0.8128" layer="16"/>
-<wire x1="37.45" y1="8.99" x2="40.12" y2="9.15" width="0.8128" layer="16"/>
-<wire x1="40.12" y1="9.15" x2="45.9375" y2="8.935" width="0.8128" layer="16"/>
-<wire x1="45.9375" y1="8.935" x2="48.4775" y2="8.935" width="0.8128" layer="16"/>
+<contactref element="U$1" pad="RST"/>
+<contactref element="U$1" pad="CH_PD"/>
+<contactref element="U$1" pad="VCC"/>
+<contactref element="U$1" pad="GPIO2"/>
+<wire x1="48.4775" y1="8.935" x2="48.4775" y2="11.475" width="0.8128" layer="16"/>
 <wire x1="48.4775" y1="8.935" x2="48.4775" y2="6.395" width="0.8128" layer="16"/>
-<wire x1="48.4775" y1="6.395" x2="48.4775" y2="3.855" width="0.8128" layer="16"/>
+<wire x1="48.4775" y1="6.395" x2="45.9375" y2="6.395" width="0.8128" layer="16"/>
+<wire x1="46" y1="22.43" x2="48.4775" y2="22.43" width="0.8128" layer="16"/>
+<wire x1="48.4775" y1="22.43" x2="48.4775" y2="11.475" width="0.8128" layer="16"/>
+<wire x1="34.81" y1="12.07" x2="34.81" y2="9.15" width="0.8128" layer="16"/>
+<wire x1="34.81" y1="9.15" x2="35.12" y2="9.15" width="0.8128" layer="16"/>
+<wire x1="35.12" y1="9.15" x2="35.12" y2="6.99" width="0.8128" layer="16"/>
+<wire x1="35.12" y1="6.99" x2="38.04" y2="6.99" width="0.8128" layer="16"/>
+<wire x1="38.04" y1="6.99" x2="38.04" y2="7.01" width="0.8128" layer="16"/>
+<wire x1="38.04" y1="7.01" x2="41.55" y2="7.01" width="0.8128" layer="16"/>
+<wire x1="41.55" y1="7.01" x2="41.55" y2="6.395" width="0.8128" layer="16"/>
+<wire x1="41.55" y1="6.395" x2="45.9375" y2="6.395" width="0.8128" layer="16"/>
 </signal>
 <signal name="GPIO0">
 <contactref element="OK1" pad="2"/>
 <contactref element="R2" pad="1"/>
-<contactref element="U$1" pad="GPIO2"/>
-<wire x1="43.07" y1="6.57" x2="27" y2="6.57" width="0.8128" layer="16"/>
-<wire x1="27" y1="6.57" x2="27" y2="10" width="0.8128" layer="16"/>
-<wire x1="27" y1="10" x2="22.13" y2="10" width="0.8128" layer="16"/>
-<wire x1="22.13" y1="10" x2="22.13" y2="10.15" width="0.8128" layer="16"/>
-<wire x1="43.07" y1="6.57" x2="45.9375" y2="6.57" width="0.8128" layer="16"/>
-<wire x1="45.9375" y1="6.57" x2="45.9375" y2="6.395" width="0.8128" layer="16"/>
+<contactref element="U$1" pad="GPIO0"/>
+<wire x1="45.9375" y1="8.935" x2="42.43" y2="8.935" width="0.8128" layer="16"/>
+<wire x1="42.43" y1="8.935" x2="42.43" y2="12.07" width="0.8128" layer="16"/>
+<wire x1="42.43" y1="12.07" x2="42.43" y2="15" width="0.8128" layer="16"/>
+<wire x1="42.43" y1="15" x2="28" y2="15" width="0.8128" layer="16"/>
+<wire x1="28" y1="15" x2="28" y2="10.15" width="0.8128" layer="16"/>
+<wire x1="28" y1="10.15" x2="22.13" y2="10.15" width="0.8128" layer="16"/>
 </signal>
 <signal name="N$2">
@@
 <contactref element="C5" pad="2"/>
 <contactref element="C3" pad="-"/>
-<contactref element="U$1" pad="RX"/>
-<wire x1="37.45" y1="11.53" x2="34.997353125" y2="11.538325" width="0.8128" layer="16"/>
-<wire x1="34.997353125" y1="11.538325" x2="31.96" y2="11.55" width="0.8128" layer="16"/>
-<wire x1="41.044" y1="22.38" x2="36.07" y2="22.38" width="0.8128" layer="16"/>
-<wire x1="34.997353125" y1="22.38" x2="34.997353125" y2="11.538325" width="0.8128" layer="16"/>
+<contactref element="U$1" pad="GND"/>
 <wire x1="36.07" y1="25.72" x2="36.07" y2="22.38" width="0.8128" layer="16"/>
-<wire x1="36.07" y1="22.38" x2="34.997353125" y2="22.38" width="0.8128" layer="16"/>
-<wire x1="37.45" y1="11.53" x2="45.9375" y2="11.475" width="0.8128" layer="16"/>
+<wire x1="36.07" y1="22.38" x2="41.044" y2="22.38" width="0.8128" layer="16"/>
+<wire x1="41.044" y1="22.38" x2="41.044" y2="29" width="0.8128" layer="16"/>
+<wire x1="41.044" y1="29" x2="51" y2="29" width="0.8128" layer="16"/>
+<wire x1="51" y1="29" x2="51" y2="2" width="0.8128" layer="16"/>
+<wire x1="51" y1="2" x2="46" y2="2" width="0.8128" layer="16"/>
+<wire x1="46" y1="2" x2="46" y2="3.855" width="0.8128" layer="16"/>
+<wire x1="46" y1="3.855" x2="45.9375" y2="3.855" width="0.8128" layer="16"/>
+<wire x1="45.9375" y1="3.855" x2="45.9375" y2="4.47" width="0.8128" layer="16"/>
+<wire x1="45.9375" y1="4.47" x2="41.55" y2="4.47" width="0.8128" layer="16"/>
+<wire x1="41.55" y1="4.47" x2="41.55" y2="4.45" width="0.8128" layer="16"/>
+<wire x1="41.55" y1="4.45" x2="38.04" y2="4.45" width="0.8128" layer="16"/>
 </signal>
 <signal name="N$4">
