File: TOM2015/Hardware/Tomada/tomada esp-tom.sch (EAGLE design)
At the start: 20 parts, among them K2 G5L, X1 MKDSN1,5/2-5,08, X2 MKDSN1,5/2-5,08

Commit message: Versão final do tom
Versão final do Tom com as ligações do esp corretas e o desenho correto
do componente TIL111
Parts:
- OK1: device optocoupler:H11L1M -> optocoupler2:H11L1M
Connections:
- net 3.3V: now also U$1.GPIO2, U$1.VCC; no longer U$1.GPIO0, U$1.TXD
- net GND: now also U$1.GND; no longer U$1.RXD
- net GPIO0: now also U$1.GPIO0; no longer U$1.GPIO2
Changed lines of the file:
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@@
 <part name="R1" library="resistor" deviceset="R-US_" device="0204/7" value="330"/>
 <part name="R2" library="resistor" deviceset="R-US_" device="0204/7" value="10k"/>
-<part name="OK1" library="optocoupler" deviceset="H11L*M" device="" technology="1"/>
+<part name="OK1" library="optocoupler2" deviceset="H11L*M" device="" technology="1"/>
 <part name="Q1" library="transistors" deviceset="2N700*" device="_TO92" technology="0"/>
 <part name="U$1" library="esp8266modules" deviceset="ESP01" device=""/>
@@
 <instance part="C1" gate="G$1" x="111.76" y="35.56"/>
 <instance part="D1" gate="1" x="114.3" y="68.58" rot="R90"/>
-<instance part="GND3" gate="1" x="27.94" y="-15.24"/>
+<instance part="GND3" gate="1" x="12.7" y="5.08" rot="R270"/>
 <instance part="X1" gate="-1" x="-53.34" y="96.52" rot="R180"/>
 <instance part="X1" gate="-2" x="-53.34" y="83.82" rot="R180"/>
@@
 </segment>
 <segment>
+<label x="78.74" y="0" size="1.778" layer="95"/>
+<pinref part="U$1" gate="G$1" pin="RST"/>
+<wire x1="66.04" y1="0" x2="71.12" y2="0" width="0.1524" layer="91"/>
 <pinref part="U$1" gate="G$1" pin="CH_PD"/>
+<wire x1="71.12" y1="0" x2="76.2" y2="0" width="0.1524" layer="91"/>
 <wire x1="71.12" y1="0" x2="71.12" y2="2.54" width="0.1524" layer="91"/>
 <wire x1="71.12" y1="2.54" x2="66.04" y2="2.54" width="0.1524" layer="91"/>
 <junction x="71.12" y="0"/>
-<wire x1="71.12" y1="0" x2="76.2" y2="0" width="0.1524" layer="91"/>
-<label x="78.74" y="0" size="1.778" layer="95"/>
-<pinref part="U$1" gate="G$1" pin="RST"/>
-<wire x1="71.12" y1="0" x2="66.04" y2="0" width="0.1524" layer="91"/>
-<pinref part="U$1" gate="G$1" pin="TXD"/>
-<wire x1="71.12" y1="2.54" x2="71.12" y2="5.08" width="0.1524" layer="91"/>
-<wire x1="71.12" y1="5.08" x2="66.04" y2="5.08" width="0.1524" layer="91"/>
-<junction x="71.12" y="2.54"/>
+<pinref part="U$1" gate="G$1" pin="VCC"/>
+<wire x1="71.12" y1="0" x2="71.12" y2="-2.54" width="0.1524" layer="91"/>
+<wire x1="71.12" y1="-2.54" x2="66.04" y2="-2.54" width="0.1524" layer="91"/>
 </segment>
 <segment>
@@
 </segment>
 <segment>
-<pinref part="U$1" gate="G$1" pin="GPIO0"/>
-<wire x1="33.02" y1="0" x2="25.4" y2="0" width="0.1524" layer="91"/>
-<label x="25.4" y="0" size="1.778" layer="95" rot="R180"/>
+<pinref part="U$1" gate="G$1" pin="GPIO2"/>
+<wire x1="33.02" y1="2.54" x2="25.4" y2="2.54" width="0.1524" layer="91"/>
+<label x="20.32" y="2.54" size="1.778" layer="95"/>
 </segment>
 </net>
@@
 </segment>
 <segment>
-<pinref part="U$1" gate="G$1" pin="GPIO2"/>
-<wire x1="33.02" y1="2.54" x2="25.4" y2="2.54" width="0.1524" layer="91"/>
-<label x="25.4" y="2.54" size="1.778" layer="95" rot="R180"/>
+<pinref part="U$1" gate="G$1" pin="GPIO0"/>
+<wire x1="33.02" y1="0" x2="25.4" y2="0" width="0.1524" layer="91"/>
+<label x="20.32" y="0" size="1.778" layer="95"/>
 </segment>
 </net>
@@
 <segment>
 <pinref part="GND3" gate="1" pin="GND"/>
-<wire x1="27.94" y1="-2.54" x2="27.94" y2="-12.7" width="0.1524" layer="91"/>
-<pinref part="U$1" gate="G$1" pin="RXD"/>
-<wire x1="27.94" y1="-2.54" x2="33.02" y2="-2.54" width="0.1524" layer="91"/>
+<wire x1="33.02" y1="5.08" x2="15.24" y2="5.08" width="0.1524" layer="91"/>
+<pinref part="U$1" gate="G$1" pin="GND"/>
 </segment>
 <segment>
